Commit message: renamed spot_description bundle

File: spot_gazebo_description/models/spot/model.urdf (robot description, URDF)
Before this commit: robot spot, 20 links, 19 joints
Links:
- link base_link: geometry collision mesh filename=package://spot_gazebo_description/meshes/body_collision.stl; visual mesh filename=package://spot_gazebo_description/meshes/body.dae
- link front_left_hip: geometry collision mesh filename=package://spot_gazebo_description/meshes/front_left_hip_col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; visual mesh filename=package://spot_gazebo_description/meshes/front_left_hip.dae
- link front_left_lower_leg: geometry collision mesh filename=package://spot_gazebo_description/meshes/front_left_lower_l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 scale=-1.82 0.97 0.98; visual mesh filename=package://spot_gazebo_description/meshes/front_left_lower_l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
- link front_left_upper_leg: geometry collision mesh filename=package://spot_gazebo_description/meshes/front_left_upper_l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; visual mesh filename=package://spot_gazebo_description/meshes/front_left_upper_l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
- link front_right_hip: geometry collision mesh filename=package://spot_gazebo_description/meshes/front_right_hip_co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; visual mesh filename=package://spot_gazebo_description/meshes/front_right_hip.dae
- link front_right_lower_leg: geometry collision mesh filename=package://spot_gazebo_description/meshes/front_right_lower_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 scale=-1.82 0.97 0.98; visual mesh filename=package://spot_gazebo_description/meshes/front_right_lower_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
- link front_right_upper_leg: geometry collision mesh filename=package://spot_gazebo_description/meshes/front_right_upper_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; visual mesh filename=package://spot_gazebo_description/meshes/front_right_upper_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
- link rear_left_hip: geometry collision mesh filename=package://spot_gazebo_description/meshes/rear_left_hip_coll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; visual mesh filename=package://spot_gazebo_description/meshes/rear_left_hip.dae
- link rear_left_lower_leg: geometry collision mesh filename=package://spot_gazebo_description/meshes/rear_left_lower_le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 scale=-1.82 0.97 0.98; visual mesh filename=package://spot_gazebo_description/meshes/rear_left_lower_le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
- link rear_left_upper_leg: geometry collision mesh filename=package://spot_gazebo_description/meshes/rear_left_upper_le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; visual mesh filename=package://spot_gazebo_description/meshes/rear_left_upper_le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
- link rear_right_hip: geometry collision mesh filename=package://spot_gazebo_description/meshes/rear_right_hip_col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; visual mesh filename=package://spot_gazebo_description/meshes/rear_right_hip.dae
- link rear_right_lower_leg: geometry collision mesh filename=package://spot_gazebo_description/meshes/rear_right_lower_l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 scale=-1.82 0.97 0.98; visual mesh filename=package://spot_gazebo_description/meshes/rear_right_lower_l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
- link rear_right_upper_leg: geometry collision mesh filename=package://spot_gazebo_description/meshes/rear_right_upper_l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; visual mesh filename=package://spot_gazebo_description/meshes/rear_right_upper_l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
